File: corne-chocolate/pcb/corne-chocolate.kicad_pcb (KiCad board)
At the start: 2 copper layers, 133.8 x 91.4 mm, 98 parts, among them J3 LED, P1 i2c-pin, P2 i2c-pin, SW1 SW_PUSH, SW10 SW_PUSH, SW11 SW_PUSH, SW12 SW_PUSH, SW13 SW_PUSH, SW14 SW_PUSH, SW15 SW_PUSH, SW16 SW_PUSH, SW17 SW_PUSH, SW18 SW_PUSH, SW19 SW_PUSH, SW2 SW_PUSH, SW20 SW_PUSH, SW21 SW_PUSH, SW3 SW_PUSH, SW4 SW_PUSH, SW5 SW_PUSH, SW6 SW_PUSH, SW7 SW_PUSH, SW8 SW_PUSH, SW9 SW_PUSH, U1 ProMicro

Commit message: corne-chocolate: moved I2C jumpers
Parts:
- moved JP2 1.62 mm to (188.9, 102.9)
- moved JP3 1.62 mm to (186.4, 102.9)
- moved JP4 1.62 mm to (183.9, 102.9)
- moved JP5 1.62 mm to (181.4, 102.9)
- moved JP6 1.62 mm to (188.9, 102.9)
- moved JP7 1.62 mm to (186.4, 102.9)
- moved JP8 1.62 mm to (183.9, 102.9)
- moved JP9 1.62 mm to (181.4, 102.9)
Routing:
- net GND: track 816.7 -> 822.1 mm, vias 59 -> 58
- net Net-(J2-Pad4): track 7.14 -> 3.90 mm
- net Net-(J2-Pad3): track 7.10 -> 3.86 mm
- net Net-(J2-Pad2): track 7.13 -> 3.89 mm
- net Net-(J2-Pad1): track 7.16 -> 3.92 mm

Commit message: moving tracks
Parts:
- removed ? (x9): , kbd:LEGO_HOLE
- removed G*** (x2): LOGO, kbd:corne
- RSW1: value Reset -> SW_PUSH
- renumbered TRRS to J1, OLED to J2, data to JP1
Routing:
- net row2: track 209.9 -> 208.8 mm

Commit message: changed board settings
Parts:
- added JP10: , kbd:Jumper, F.Cu at (179.1, 111.4)
- added JP11: , kbd:Jumper, B.Cu at (176.8, 111.4)
- added JP12: , kbd:Jumper, B.Cu at (179.1, 111.4)
- added JP13: , kbd:Jumper, B.Cu at (176.0, 103.5)
- added JP14: , kbd:Jumper, B.Cu at (176.0, 107.0)
- added P3: i2c-pin, kbd:1pin_conn, F.Cu at (189.6, 84.5)
- added P4: i2c-pin, kbd:1pin_conn, F.Cu at (180.7, 83.2)
- added P5: i2c-pin, kbd:1pin_conn, F.Cu at (180.7, 80.7)
- added P6: i2c-pin, kbd:1pin_conn, F.Cu at (189.6, 81.9)
- JP1: footprint kbd:JPC2 -> kbd:Jumper
- moved JP1 4.55 mm to (176.8, 111.4)
Connections:
- J1 pad A: Net-(J1-PadA) -> /A
- J1 pad B: Net-(J1-PadB) -> /B
- JP1 pad 1: data -> /TX
- JP1 pad 2: Net-(J1-PadB) -> /A
- P1 pad 1: Net-(J1-PadA) -> /A
- P2 pad 1: Net-(J1-PadB) -> /B
- U1 pad 1: LED -> /TX
- U1 pad 12: Net-(U1-Pad12) -> /BL
- U1 pad 2: data -> /RX
- U1 pad 3: GND -> Net-(U1-Pad3)
Routing:
- net /TX: track 0.00 -> 62.2 mm, vias 0 -> 3
- net /RX: track 0.00 -> 57.0 mm, vias 0 -> 3
- net data: track 55.9 -> 0.00 mm, vias 4 -> 0
- net /B: track 0.00 -> 24.5 mm
- net /BL: track 0.00 -> 20.1 mm
- net Net-(J1-PadB): track 19.0 -> 0.00 mm, vias 1 -> 0
- net Net-(U1-Pad12): track 18.9 -> 0.00 mm
- net /A: track 0.00 -> 16.1 mm
- net SCL: track 46.3 -> 60.2 mm, vias 2 -> 3
- net GND: track 822.1 -> 808.2 mm, vias 58 -> 57
- net LED: track 79.9 -> 68.1 mm, vias 10 -> 8
- net Net-(J1-PadA): track 10.3 -> 0.00 mm
- net reset: track 41.7 -> 45.4 mm
- net col0: track 255.1 -> 257.2 mm, vias 12 -> 10
- net SDA: track 55.4 -> 54.3 mm
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Other:
- rule pad_to_mask_clearance: 0.2 -> 0.051
